File: mSeguier/mSeguier.kicad_sch (KiCad schematic)
At the start: 12 parts, among them J1 Bornier 3 vis, K1 Finder 30.22.7.005, Q1 BS270, U1 MuseLab nanoESP32-C6, U2 BH1750 (GY-302), U3 BMP280 (GY-BMP280), U4 Capteur gaz MQ, U5 RC522 RFID, U6 ILI9341 2.4" + XPT2046

Commit message: KiCad mSeguier : référence complète du relais K1 (Finder 30.22.7.005.0010)
Co-Authored-By: Claude Opus 5.5 (1M context) <noreply@anthropic.com>
Claude-Session: https://claude.ai/code/session_018mRuxxBd7hy4gYvrch8s8D
Parts:
- K1: value Finder 30.22.7.005 -> Finder 30.22.7.005.0010
Changed lines of the file:
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@@
 			)
 		)
-		(property "Value" "Finder 30.22.7.005"
+		(property "Value" "Finder 30.22.7.005.0010"
 			(at 250.19 58.42 0)
 			(show_name no)
