File: mSeguier/mSeguier.kicad_pcb (KiCad board)
At the start: 2 copper layers, 170 x 90 mm, 14 parts, among them J1 Bornier 3 vis, K1 Finder 30.22.7.005, Q1 BS270, U1 MuseLab nanoESP32-C6, U2 BH1750 (GY-302), U3 BMP280 (GY-BMP280), U4 Capteur gaz MQ, U5 RC522 RFID, U6 ILI9341 2.4" + XPT2046

Commit message: KiCad mSeguier : PCB au format KiCad 9, recalé sur le schéma (bobine du relais câblée)
Le PCB était au format KiCad 10, illisible par KiCad 9 sous Windows.
Il est reconstruit en KiCad 9 avec le schéma enregistré par l'utilisateur
(réseau de la bobine renommé Net-(D1-A), gardé en classe Fort courant),
re-routé, plans de masse re-remplis, Gerber et perçage régénérés.
DRC KiCad 9 et 10 : 0 erreur, 0 avertissement, parité schéma OK.

Co-Authored-By: Claude Opus 5.5 (1M context) <noreply@anthropic.com>
Claude-Session: https://claude.ai/code/session_018mRuxxBd7hy4gYvrch8s8D
Connections:
- net /RELAY_COIL renamed Net-(D1-A)
Routing:
- net +3V3: track 269.7 -> 208.6 mm, vias 1 -> 0
- net GND: track 399.8 -> 430.6 mm
- net /TOUCH_CS: track 54.3 -> 37.4 mm, vias 1 -> 0
- net /TFT_RST: track 84.4 -> 98.9 mm
- net +5V: track 171.4 -> 159.3 mm, vias 2 -> 0
- net Net-(D1-A): track 35.5 -> 24.0 mm
- net /TFT_DC: track 80.8 -> 91.9 mm
- net /SPI_MOSI: track 164.6 -> 158.1 mm, vias 0 -> 3
- net /SPI_SCK: track 153.1 -> 159.0 mm
- net /MQ_AO: track 88.8 -> 93.0 mm
- net /TFT_CS: track 87.5 -> 90.8 mm
- net /SPI_MISO: track 148.6 -> 151.6 mm, vias 0 -> 1
- net /RELAY_CMD: track 113.2 -> 110.7 mm, vias 2 -> 0
- net /RFID_RST: track 75.6 -> 75.3 mm, vias 0 -> 1
- net /RFID_CS: vias 0 -> 1

Commit message: KiCad mSeguier : retour au routage précédent, schéma de l'utilisateur conservé
Mêmes pistes et vias que la version KiCad 10 d'avant f8243e8, reportées en
format KiCad 9 sur le schéma modifié par l'utilisateur (bobine du relais
câblée, réseau Net-(D1-A)). DRC KiCad 9 et 10 : 0 erreur, 0 avertissement.

Co-Authored-By: Claude Opus 5.5 (1M context) <noreply@anthropic.com>
Claude-Session: https://claude.ai/code/session_018mRuxxBd7hy4gYvrch8s8D
Routing:
- net +3V3: track 208.6 -> 269.7 mm, vias 0 -> 1
- net GND: track 430.6 -> 399.8 mm
- net /TOUCH_CS: track 37.4 -> 54.3 mm, vias 0 -> 1
- net /TFT_RST: track 98.9 -> 84.4 mm
- net +5V: track 159.3 -> 171.4 mm, vias 0 -> 2
- net Net-(D1-A): track 24.0 -> 35.5 mm
- net /TFT_DC: track 91.9 -> 80.8 mm
- net /SPI_MOSI: track 158.1 -> 164.6 mm, vias 3 -> 0
- net /SPI_SCK: track 159.0 -> 153.1 mm
- net /MQ_AO: track 93.0 -> 88.8 mm
- net /TFT_CS: track 90.8 -> 87.5 mm
- net /SPI_MISO: track 151.6 -> 148.6 mm, vias 1 -> 0
- net /RELAY_CMD: track 110.7 -> 113.2 mm, vias 0 -> 2
- net /RFID_RST: track 75.3 -> 75.6 mm, vias 1 -> 0
- net /RFID_CS: vias 1 -> 0

Commit message: KiCad mSeguier : référence complète du relais K1 (Finder 30.22.7.005.0010)
Co-Authored-By: Claude Opus 5.5 (1M context) <noreply@anthropic.com>
Claude-Session: https://claude.ai/code/session_018mRuxxBd7hy4gYvrch8s8D
Parts:
- K1: value Finder 30.22.7.005 -> Finder 30.22.7.005.0010
Changed lines of the file:
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@@
 			)
 		)
-		(property "Value" "Finder 30.22.7.005"
+		(property "Value" "Finder 30.22.7.005.0010"
 			(at 8.4 2.4 0)
 			(layer "F.Fab")
